Commit message: Add inertial macros and define robot structure with wheels and chassis

File: description/robot_core.xacro (robot description, xacro)
@@ -1,21 +1,70 @@
 <?xml version="1.0"?>
 <robot xmlns:xacro="http://www.ros.org/wiki/xacro"  >
+    <xacro:include filename="inertial_macros.xacro"/>
     <material name="white">  <!-- Define a material named white -->
-    <color rgba="1 1 1 1"/>
+        <color rgba="1 1 1 1"/>
     </material>
     <material name="black">  <!-- Define a material named black -->
-    <color rgba="0 0 0 1"/>
+        <color rgba="0 0 0 1"/>
     </material>
     <material name="red">   <!-- Define a material named red -->
-    <color rgba="1 0 0 1"/>
+        <color rgba="1 0 0 1"/>
     </material>
     <material name="blue">  <!-- Define a material named blue -->
-    <color rgba="0 0 1 1"/>
+        <color rgba="0 0 1 1"/>
     </material>
     <material name="green"> <!-- Define a material named green -->
-    <color rgba="0 1 0 1"/>
+        <color rgba="0 1 0 1"/>
     </material>
+<!-- Define a link named base_link-->
     <link name="base_link">
     </link>
+    <!-- Define a link named left_wheel -->
+    <joint name="left_wheel_joint" type="continuous">
+        <parent link="base_link"/>
+        <child link="left_wheel"/>
+        <origin xyz="0 0.175 0" rpy="-${pi/2} 0 0"/>
+        <axis xyz="0 0 1"/>
+    </joint>
+    <link name="left_wheel">
+        <visual>
+            <geometry>
+                <cylinder radius="0.05" length="0.04"/>
+            </geometry>
+            <material name="blue"/>
+        </visual>
+        <collision>
+            <geometry>
+                <cylinder radius="0.05" length="0.04"/>
+            </geometry>
+        </collision>
+        <xacro:inertial_cylinder mass="0.1" radius="0.05" length="0.04">
+            <origin xyz="0 0 0" rpy="0 0 0"/>
+        </xacro:inertial_cylinder>
+    </link>
+    <!-- Define a link named right_wheel -->
+    <joint name="right_wheel_joint" type="continuous">
+        <parent link="base_link"/>
+        <child link="right_wheel"/>
+        <origin xyz="0 -0.175 0" rpy="${pi/2} 0 0"/>
+        <axis xyz="0 0 -1"/>
+    </joint>
+    <link name="right_wheel">
+        <visual>
+            <geometry>
+                <cylinder radius="0.05" length="0.04"/>
+            </geometry>
+            <material name="blue"/>
+        </visual>
+        <collision>
+            <geometry>
+                <cylinder radius="0.05" length="0.04"/>
+            </geometry>
+        </collision>
+        <xacro:inertial_cylinder mass="0.1" radius="0.05" length="0.04">
+            <origin xyz="0 0 0" rpy="0 0 0"/>
+        </xacro:inertial_cylinder>
+    </link>
+<!-- Define a link named chassis -->
     <joint name="chassis_joint" type="fixed">
         <origin xyz="-0.1 0 0"/>
@@ -23,12 +72,43 @@
         <child link="chassis"/>
     </joint>
-    <link name="chassis">  <!-- Define a link named chassis -->
-    <visual>
-        <origin xyz="0.15 0 0.075"/>
-        <geometry>
-            <box size="0.3 0.3 0.15"/>
-        </geometry>
-        <material name="white"/>
-    </visual>
+    <link name="chassis">
+        <visual>
+            <origin xyz="0.15 0 0.075"/>
+            <geometry>
+                <box size="0.3 0.3 0.15"/>
+            </geometry>
+            <material name="white"/>
+        </visual>
+        <collision>
+            <origin xyz="0.15 0 0.075"/>
+            <geometry>
+                <box size="0.3 0.3 0.15"/>
+            </geometry>
+        </collision>
+        <xacro:inertial_box mass="0.5" x="0.3" y="0.3" z="0.15">
+            <origin xyz="0.15 0 0.075" rpy ="0 0 0"/>
+        </xacro:inertial_box>
+    </link>
+    <!--caster wheel -->
+    <joint name="caster_wheel_joint" type="fixed">
+        <parent link="chassis"/>
+        <child link="caster_wheel"/>
+        <origin xyz="0.24 0 0"/>
+    </joint>
+    <link name="caster_wheel">
+        <visual>
+            <geometry>
+                <sphere radius="0.05"/>
+            </geometry>
+            <material name="red"/>
+        </visual>
+        <collision>
+            <geometry>
+                <sphere radius="0.05"/>
+            </geometry>
+        </collision>
+        <xacro:inertial_sphere mass="0.1" radius="0.05">
+            <origin xyz="0 0 0" rpy="0 0 0"/>
+        </xacro:inertial_sphere>
     </link>
 </robot>
